Commit message: arm

File: urdf/omni.urdf (robot description, URDF)
Before this commit: robot omni, 9 links, 8 joints
Joints:
- joint joint_arm_1: limit lower=0 upper=3.14 effort=10 velocity=10 -> lower=0 upper=3.14 effort=100 velocity=10
- joint joint_arm_2: limit lower=-1.57 upper=0 effort=10 velocity=10 -> lower=-1.57 upper=0 effort=100 velocity=10

Commit message: control

File: urdf/omni.urdf (robot description, URDF)
Before this commit: robot omni, 9 links, 8 joints
Joints:
- joint joint_arm_2: limit lower=-1.57 upper=0 effort=100 velocity=10 -> lower=-1.57 upper=1.57 effort=100 velocity=10

Commit message: update

File: urdf/omni.urdf (robot description, URDF)
Before this commit: robot omni, 9 links, 8 joints
Joints:
- joint joint_arm_1: limit lower=0 upper=3.14 effort=100 velocity=10 -> lower=-3.14 upper=3.14 effort=100 velocity=10
- joint joint_arm_2: limit lower=-1.57 upper=1.57 effort=100 velocity=10 -> lower=-1.57 upper=0.79 effort=100 velocity=10
